File: PCB/PCB- Sensing/MicroMouse Sensor .kicad_sch (KiCad schematic)
At the start: 43 parts, among them J1 Conn_02x14_Odd_Even, Q1 C2150, Q2 C2150, Q3 C2150, Q4 C2150, Q5 C2150, Q6 C2150, U1 OP07, U2 OP07, U3 OP07

Commit message: Sensor Documents Update
Connections:
- net PE14: now also R1.1, R2.1, R9.1
- net PE15: no longer R1.1, R11.1, R2.1, R5.1, R7.1, R9.1
- net PE8: now also R11.1, R7.1
- net PE9: now also R5.1
Changed lines of the file:
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@@
   (title_block
     (title "Micro Mouse Sensor")
-    (date "2024-03-20")
-    (rev "v4.0")
+    (date "2024-05-10")
+    (rev "v5.0")
     (company "University of Cape Town")
     (comment 1 "EEE3088F")
@@
     )
   )
-  (global_label "PE15" (shape input) (at 96.52 130.81 0) (fields_autoplaced)
+  (global_label "PE14" (shape input) (at 96.52 130.81 0) (fields_autoplaced)
     (effects (font (size 1.27 1.27)) (justify left))
     (property "Intersheetrefs" "${INTERSHEET_REFS}" (at 104.2638 130.81 0)
@@
     )
   )
-  (global_label "PE15" (shape input) (at 171.45 66.04 180) (fields_autoplaced)
+  (global_label "PE14" (shape input) (at 171.45 66.04 180) (fields_autoplaced)
     (effects (font (size 1.27 1.27)) (justify right))
     (property "Intersheetrefs" "${INTERSHEET_REFS}" (at 163.7062 66.04 0)
@@
     )
   )
-  (global_label "PE15" (shape input) (at 163.83 127 0) (fields_autoplaced)
-    (effects (font (size 1.27 1.27)) (justify left))
-    (property "Intersheetrefs" "${INTERSHEET_REFS}" (at 171.5738 127 0)
+  (global_label "PE8" (shape input) (at 163.83 127 0) (fields_autoplaced)
+    (effects (font (size 1.27 1.27)) (justify left))
+    (property "Intersheetrefs" "${INTERSHEET_REFS}" (at 170.3643 127 0)
       (effects (font (size 1.27 1.27)) (justify left) hide)
     )
@@
     )
   )
-  (global_label "PE15" (shape input) (at 224.79 67.31 180) (fields_autoplaced)
-    (effects (font (size 1.27 1.27)) (justify right))
-    (property "Intersheetrefs" "${INTERSHEET_REFS}" (at 217.0462 67.31 0)
-      (effects (font (size 1.27 1.27)) (justify right) hide)
-    )
-  )
-  (global_label "PE15" (shape input) (at 119.38 64.77 180) (fields_autoplaced)
+  (global_label "PE9" (shape input) (at 224.79 67.31 180) (fields_autoplaced)
+    (effects (font (size 1.27 1.27)) (justify right))
+    (property "Intersheetrefs" "${INTERSHEET_REFS}" (at 218.2557 67.31 0)
+      (effects (font (size 1.27 1.27)) (justify right) hide)
+    )
+  )
+  (global_label "PE14" (shape input) (at 119.38 64.77 180) (fields_autoplaced)
     (effects (font (size 1.27 1.27)) (justify right))
     (property "Intersheetrefs" "${INTERSHEET_REFS}" (at 111.6362 64.77 0)
@@
     )
   )
-  (global_label "PE15" (shape input) (at 22.86 130.81 0) (fields_autoplaced)
-    (effects (font (size 1.27 1.27)) (justify left))
-    (property "Intersheetrefs" "${INTERSHEET_REFS}" (at 30.6038 130.81 0)
-      (effects (font (size 1.27 1.27)) (justify left) hide)
-    )
+  (global_label "PE8" (shape input) (at 22.86 130.81 0) (fields_autoplaced)
+    (effects (font (size 1.27 1.27)) (justify left))
+    (property "Intersheetrefs" "${INTERSHEET_REFS}" (at 29.3943 130.81 0)
+      (effects (font (size 1.27 1.27)) (justify left) hide)
+    )
